Commit message: updated urdf

File: src/ackermann_gazebo/urdf/bot.xacro (robot description, xacro)
@@ -1,9 +1,6 @@
 <?xml version="1.0"?>
 <robot xmlns:xacro="http://www.ros.org/wiki/xacro">
-  <!-- ===================== -->
-  <!-- PROPERTIES (UPDATED) -->
-  <!-- ===================== -->
   <!-- Chassis -->
-  <xacro:property name="body_mass" value="25.0" />
+  <xacro:property name="body_mass" value="1.58" />
   <xacro:property name="body_width" value="0.355" />   <!-- Y -->
   <xacro:property name="body_length" value="0.160" /> <!-- Z -->
@@ -12,6 +9,6 @@
   <xacro:property name="wheel_radius" value="0.055" />
   <xacro:property name="wheel_thickness" value="0.070" />
-  <xacro:property name="wheel_mass" value="3.0" />
-  <xacro:property name="steering_mass" value="0.01" />
+  <xacro:property name="wheel_mass" value="0.12" />
+  <xacro:property name="steering_mass" value="0.02" />
   <!-- ===================== -->
   <!-- BASE -->
@@ -31,6 +28,6 @@
   <link name="chassis_link">
     <inertial>
-      <origin xyz="0 0 0" rpy="0 0 0" />
-      <mass value="25.0" />
+      <origin xyz="0.0374140021041951 -0.000373005187591258 -0.0771282894414029" rpy="0 0 0" />
+      <mass value="1.58" />
       <inertia
         ixx="${body_mass/12 * (body_width*body_width + body_length*body_length)}"
@@ -65,5 +62,5 @@
   <link name="fr_left_steer_link">
     <inertial>
-      <origin xyz="0 0 0" rpy="0 0 0" />
+      <origin xyz="-0.0002776492198312 0.0163539773588368 4.97346169803237E-09" rpy="0 0 0" />
       <mass value="${steering_mass}" />
       <inertia
@@ -74,4 +71,19 @@
         izz="${steering_mass/2 * wheel_radius*wheel_radius}" />
     </inertial>
+    <visual>
+      <origin xyz="0.0 0.0 0.0" rpy="1.570795 0.0 0.0"/>
+      <geometry>
+        <cylinder length="0.001" radius="0.01"/>
+      </geometry>
+      <material name="">
+        <color rgba="0.0 0.0 0.0 1.0"/>
+      </material>
+    </visual>
+    <collision>
+      <origin xyz="0.0 0.0 0.0" rpy="1.570795 0.0 0.0"/>
+      <geometry>
+        <cylinder length="0.001" radius="0.01"/>
+      </geometry>
+    </collision>
   </link>
   <joint name="fr_left_steer_joint" type="revolute">
@@ -84,5 +96,5 @@
   <link name="fr_left_wheel_link">
     <inertial>
-      <origin xyz="0 0 0" rpy="0 0 0" />
+      <origin xyz="-3.5837499634539E-10 4.97346158701006E-09 -0.016356334080185" rpy="0 0 0" />
       <mass value="${wheel_mass}" />
       <inertia
@@ -97,6 +109,10 @@
         <cylinder radius="${wheel_radius}" length="${wheel_thickness}" />
       </geometry>
-    </visual>
-    <collision>
+      <material name="">
+        <color rgba="0.223529411764706 0.223529411764706 0.223529411764706 1" />
+      </material>
+    </visual>
+    <collision>
+      <origin xyz="0 0 0" rpy="0 0 0" />
       <geometry>
         <cylinder radius="${wheel_radius}" length="${wheel_thickness}" />
@@ -110,4 +126,5 @@
     <axis xyz="0 0 -1" />
     <dynamics friction="0.8" damping="0.5" />
+    <limit lower="-3.14159" upper="3.14159" effort="200" velocity="-1" />
   </joint>
   <!-- ===================== -->
@@ -116,5 +133,5 @@
   <link name="fr_right_steer_link">
     <inertial>
-      <origin xyz="0 0 0" rpy="0 0 0" />
+      <origin xyz="0.000274981985673328 -0.0163540222836661 -3.24802407192237E-11" rpy="0 0 0" />
       <mass value="${steering_mass}" />
       <inertia
@@ -125,4 +142,19 @@
         izz="${steering_mass/2 * wheel_radius*wheel_radius}" />
     </inertial>
+    <visual>
+      <origin xyz="0.0 0.0 0.0" rpy="1.570795 0.0 0.0"/>
+      <geometry>
+        <cylinder length="0.001" radius="0.01"/>
+      </geometry>
+      <material name=" ">
+        <color rgba="0.0 0.0 0.0 1.0"/>
+      </material>
+    </visual>
+    <collision>
+      <origin xyz="0.0 0.0 0.0" rpy="1.570795 0.0 0.0"/>
+      <geometry>
+        <cylinder length="0.001" radius="0.01"/>
+      </geometry>
+    </collision>
   </link>
   <joint name="fr_right_steer_joint" type="revolute">
@@ -134,9 +166,27 @@
   </joint>
   <link name="fr_right_wheel_link">
-    <visual>
-      <geometry>
-        <cylinder radius="${wheel_radius}" length="${wheel_thickness}" />
-      </geometry>
-    </visual>
+        <inertial>
+            <origin xyz="0.00027498198567355 3.24801296969213E-11 -0.0163540222836661" rpy="0 0 0" />
+            <mass value="${wheel_mass}" />
+            <inertia
+                ixx="${wheel_mass/12*(3*wheel_radius*wheel_radius + wheel_thickness*wheel_thickness)}"
+                ixy="0" ixz="0"
+                iyy="${wheel_mass/12*(3*wheel_radius*wheel_radius + wheel_thickness*wheel_thickness)}"
+                iyz="0" izz="${wheel_mass/2 * wheel_radius*wheel_radius}" />
+        </inertial>
+        <visual>
+            <geometry>
+                <cylinder radius="${wheel_radius}" length="${wheel_thickness}" />
+            </geometry>
+            <material name="">
+                <color rgba="0.223529411764706 0.223529411764706 0.223529411764706 1" />
+            </material>
+        </visual>
+        <collision>
+            <origin xyz="0 0 0" rpy="0 0 0" />
+            <geometry>
+                <cylinder radius="${wheel_radius}" length="${wheel_thickness}" />
+            </geometry>
+        </collision>
   </link>
   <joint name="fr_right_wheel_joint" type="continuous">
@@ -146,9 +196,38 @@
     <axis xyz="0 0 1" />
     <dynamics friction="0.8" damping="0.5" />
+    <limit lower="-3.14159" upper="3.14159" effort="200" velocity="-1" />
   </joint>
   <!-- ===================== -->
   <!-- REAR WHEELS -->
   <!-- ===================== -->
-  <joint name="re_left_wheel_joint" type="continuous">
+  <!-- REAR LEFT WHEEL -->
+<link name="re_left_wheel_link">
+    <inertial>
+        <origin xyz="1.245E-09 1.7252E-06 -0.010284" rpy="0 0 0" />
+        <mass value="${wheel_mass}" />
+        <inertia
+            ixx="${wheel_mass/12*(3*wheel_radius*wheel_radius + wheel_thickness*wheel_thickness)}"
+            ixy="0" ixz="0"
+            iyy="${wheel_mass/12*(3*wheel_radius*wheel_radius + wheel_thickness*wheel_thickness)}"
+            iyz="0"
+            izz="${wheel_mass/2 * wheel_radius*wheel_radius}" />
+    </inertial>
+    <visual>
+        <origin xyz="0 0 0" rpy="0 0 0" />
+        <geometry>
+            <cylinder radius="${wheel_radius}" length="${wheel_thickness}" />
+        </geometry>
+        <material name="">
+            <color rgba="0.37647 0.37647 0.37647 1" />
+        </material>
+    </visual>
+    <collision>
+        <origin xyz="0 0 0" rpy="0 0 0" />
+        <geometry>
+            <cylinder radius="${wheel_radius}" length="${wheel_thickness}" />
+        </geometry>
+    </collision>
+</link>
+<joint name="re_left_wheel_joint" type="continuous">
     <parent link="chassis_link" />
     <child link="re_left_wheel_link" />
@@ -156,6 +235,35 @@
     <axis xyz="0 0 -1" />
     <dynamics friction="0.8" damping="0.5" />
-  </joint>
-  <joint name="re_right_wheel_joint" type="continuous">
+    <limit lower="-3.14159" upper="3.14159" effort="70" velocity="-1" />
+</joint>
+<!-- REAR RIGHT WHEEL -->
+<link name="re_right_wheel_link">
+    <inertial>
+        <origin xyz="0 0 0" rpy="0 0 0" />
+        <mass value="${wheel_mass}" />
+        <inertia
+            ixx="${wheel_mass/12*(3*wheel_radius*wheel_radius + wheel_thickness*wheel_thickness)}"
+            ixy="0" ixz="0"
+            iyy="${wheel_mass/12*(3*wheel_radius*wheel_radius + wheel_thickness*wheel_thickness)}"
+            iyz="0"
+            izz="${wheel_mass/2 * wheel_radius*wheel_radius}" />
+    </inertial>
+    <visual>
+        <origin xyz="0 0 0" rpy="0 0 0" />
+        <geometry>
+            <cylinder radius="${wheel_radius}" length="${wheel_thickness}" />
+        </geometry>
+        <material name="">
+            <color rgba="0.37647 0.37647 0.37647 1" />
+        </material>
+    </visual>
+    <collision>
+        <origin xyz="0 0 0" rpy="0 0 0" />
+        <geometry>
+            <cylinder radius="${wheel_radius}" length="${wheel_thickness}" />
+        </geometry>
+    </collision>
+</link>
+<joint name="re_right_wheel_joint" type="continuous">
     <parent link="chassis_link" />
     <child link="re_right_wheel_link" />
@@ -163,14 +271,31 @@
     <axis xyz="0 0 1" />
     <dynamics friction="0.8" damping="0.5" />
-  </joint>
+    <limit lower="-3.14159" upper="3.14159" effort="70" velocity="-1" />
+</joint>
   <!-- ===================== -->
   <!-- LiDAR -->
   <!-- ===================== -->
   <link name="laser_link">
+    <inertial>
+        <origin xyz="0 0 0" rpy="0 0 0"/>
+        <mass value="0.2"/>
+        <inertia ixx="0.0001" ixy="0.0" ixz="0.0"
+                    iyy="0.0001" iyz="0.0"
+                    izz="0.0001"/>
+    </inertial>
     <visual>
       <geometry>
         <cylinder radius="0.07" length="0.05"/>
       </geometry>
-    </visual>
+      <material name="">
+                <color rgba="0.1 0.1 0.1 1"/>
+      </material>
+    </visual>
+     <collision>
+        <origin xyz="0 0 0" rpy="0 0 0"/>
+        <geometry>
+            <cylinder radius="0.07" length="0.05"/>
+        </geometry>
+    </collision>
   </link>
   <joint name="laser_joint" type="fixed">

File: src/ackermann_gazebo/urdf/gz_ackermann_core.xacro (robot description, xacro)
@@ -115,4 +115,5 @@
         <plugin filename="gz-sim-joint-state-publisher-system"
             name="gz::sim::systems::JointStatePublisher">
+            <topic>joint_states</topic>
             <update_rate>100</update_rate>
             <joint_name>fr_right_steer_joint</joint_name>

File: src/ackermann_gazebo/urdf/vehicle.urdf.xacro (robot description, xacro)
@@ -3,6 +3,6 @@
 <robot xmlns:xacro="http://www.ros.org/wiki/xacro"  name="bot_ackermann">
     <!-- Physical Description -->
-    <xacro:include filename="bot.xacro" />
+    <xacro:include filename="bot_sample.xacro" />
     <!-- Simulation -->
-    <xacro:include filename="gz_ackermann_core.xacro" />
+    <!--<xacro:include filename="gz_ackermann_core.xacro" /> -->
 </robot>
