Commit message: map file added

File: src/ackermann_gazebo/urdf/bot_sample.xacro (robot description, xacro)
@@ -16,5 +16,5 @@
     <!-- max steering = 45 deg -->
     <xacro:property name="max_steering_angle" value="${pi/4}" />
-    <xacro:property name="lidar_radius" value="0.070" />
+    <xacro:property name="lidar_radius" value="0.035" />
     <xacro:property name="lidar_height" value="0.055" />
     <xacro:property name="lidar_mass" value="0.05" />
@@ -295,5 +295,5 @@
     <!-- LIDAR LINK -->
     <!-- ================================ -->
-    <link name="laser_link">
+    <link name="bot_ackermann/base_footprint/gpu_lidar">
         <inertial>
             <origin xyz="0 0 0" rpy="0 0 0" />
@@ -324,5 +324,5 @@
     <joint name="laser_joint" type="fixed">
         <parent link="chassis_link" />
-        <child link="laser_link" />
+        <child link="bot_ackermann/base_footprint/gpu_lidar" />
         <!-- LiDAR at front edge + its radius, sitting on top surface -->
         <origin xyz=" 0.1 0.0 ${body_height/2 + lidar_height/2}" rpy="0 0 0" />
@@ -402,9 +402,9 @@
     </gazebo>
     <!-- LiDAR -->
-    <gazebo reference="laser_link">
-        <material>Gazebo/Black</material>
-        <sensor name="gpu_lidar" type="gpu_lidar">
-            <pose>0 0 0 0 0 0</pose>
+    <gazebo reference="bot_ackermann/base_footprint/gpu_lidar">
+        <sensor type="gpu_lidar" name="gpu_lidar">
+            <pose relative_to='bot_ackermann/base_footprint/gpu_lidar'>0 0 0 0 0 0</pose>
             <visualize>true</visualize>
+            <topic>scan</topic>
             <update_rate>10</update_rate>
             <always_on>true</always_on>
@@ -419,5 +419,5 @@
                 </scan>
                 <range>
-                    <min>0.3</min>
+                    <min>0.15</min>
                     <max>12.0</max>
                     <resolution>0.01</resolution>
@@ -429,6 +429,4 @@
                 </noise>
             </lidar>
-            <topic>/scan</topic>
-            <frame_id>laser_link</frame_id>
         </sensor>
     </gazebo>
@@ -473,16 +471,18 @@
             <max_velocity>1</max_velocity>
             <!-- Steering limits -->
-            <max_steer>${max_steering_angle}</max_steer>
-            <max_steering_angle>1.570796</max_steering_angle>
+            <steering_limit>${max_steering_angle}</steering_limit>
             <!-- Command and odometry topics -->
             <topic>/cmd_vel</topic>
+            <tf_topic>/tf</tf_topic>
             <odom_topic>/odom</odom_topic>
-            <odom_frame>odom</odom_frame>
-            <robot_base_frame>base_footprint</robot_base_frame>
-            <!-- Publishing options -->
-            <publish_odom>true</publish_odom>
-            <publish_odom_tf>true</publish_odom_tf>
-            <publish_wheel_tf>true</publish_wheel_tf>
+            <frame_id>odom</frame_id>
+            <child_frame_id>base_footprint</child_frame_id>
+            <odom_publish_frequency>50</odom_publish_frequency>
         </plugin>
     </gazebo>
+    <gazebo>
+        <plugin filename="gz-sim-sensors-system" name="gz::sim::systems::Sensors">
+            <render_engine>ogre2</render_engine>
+        </plugin>
+  </gazebo>
 </robot>

Commit message: urdf changes

File: src/ackermann_gazebo/urdf/bot_sample.xacro (robot description, xacro)
@@ -81,5 +81,5 @@
     <link name="fr_left_steer_link">
         <inertial>
-            <origin xyz="0 0 0" rpy="0 0 0" />
+            <origin xyz="0 0 0" rpy="${pi/2} 0 0" />
             <mass value="${steering_mass}" />
             <inertia
@@ -92,5 +92,5 @@
         <!-- Simple visual so it shows in RViz/Gazebo -->
         <visual>
-            <origin xyz="0 0 0" rpy="0 0 0" />
+            <origin xyz="0 0 0" rpy="${pi/2} 0 0" />
             <geometry>
                 <cylinder radius="0.01" length="0.03"/>
@@ -100,4 +100,10 @@
             </material>
         </visual>
+        <collision>
+            <origin xyz="0 0 0" rpy="${pi/2} 0 0" />
+            <geometry>
+                <cylinder radius="0.01" length="0.03"/>
+            </geometry>
+        </collision>
     </link>
     <joint name="fr_left_steer_joint" type="revolute">
@@ -106,5 +112,6 @@
         <origin xyz="${front_axle_offset} ${half_track_width} ${-body_height/2}" rpy="0 0 0" />
         <axis xyz="0 0 1" />
-        <limit upper="${max_steering_angle}" lower="${-max_steering_angle}" effort="10.0" velocity="5.0" />
+        <limit upper="${max_steering_angle}" lower="${-max_steering_angle}" effort="10.0" velocity="2.0" />
+        <dynamics damping="0.1" friction="0.1"/>
     </joint>
     <!-- ================================ -->
@@ -113,5 +120,5 @@
     <link name="fr_left_wheel_link">
         <inertial>
-            <origin xyz="0 0 0" rpy="0 0 0" />
+            <origin xyz="0 0 0" rpy="${pi/2} 0 0" />
             <mass value="${wheel_mass}" />
             <inertia
@@ -123,5 +130,5 @@
         </inertial>
         <visual>
-            <origin xyz="0 0 0" rpy="0 0 0" />
+            <origin xyz="0 0 0" rpy="${pi/2} 0 0" />
             <geometry>
                 <cylinder radius="${wheel_radius}" length="${wheel_thickness}" />
@@ -132,5 +139,5 @@
         </visual>
         <collision>
-            <origin xyz="0 0 0" rpy="0 0 0" />
+            <origin xyz="0 0 0" rpy="${pi/2} 0 0" />
             <geometry>
                 <cylinder radius="${wheel_radius}" length="${wheel_thickness}" />
@@ -141,8 +148,8 @@
         <parent link="fr_left_steer_link" />
         <child link="fr_left_wheel_link" />
-        <origin xyz="0 0 0" rpy="${pi/2} 0 0" />
-        <axis xyz="0 0 -1" />
-        <dynamics friction="0.8" damping="0.5" />
-        <limit lower="-3.14159" upper="3.14159" effort="70" velocity="-1" />
+        <origin xyz="0 0 0" rpy="0 0 0" />
+        <axis xyz="0 1 0" />
+        <dynamics friction="0.1" damping="0.1" />
+        <limit lower="-3.14159" upper="3.14159" effort="70" velocity="50" />
     </joint>
     <!-- ================================ -->
@@ -151,5 +158,5 @@
     <link name="fr_right_steer_link">
         <inertial>
-            <origin xyz="0 0 0" rpy="0 0 0" />
+            <origin xyz="0 0 0" rpy="${pi/2} 0 0" />
             <mass value="${steering_mass}" />
             <inertia
@@ -162,5 +169,5 @@
         <!-- Simple visual so it shows in RViz/Gazebo -->
         <visual>
-            <origin xyz="0 0 0" rpy="0 0 0" />
+            <origin xyz="0 0 0" rpy="${pi/2} 0 0" />
             <geometry>
                 <cylinder radius="0.01" length="0.03"/>
@@ -170,4 +177,10 @@
             </material>
         </visual>
+        <collision>
+            <origin xyz="0 0 0" rpy="${pi/2} 0 0" />
+            <geometry>
+                <cylinder radius="0.01" length="0.03"/>
+            </geometry>
+        </collision>
     </link>
     <joint name="fr_right_steer_joint" type="revolute">
@@ -176,5 +189,6 @@
         <origin xyz="${front_axle_offset} ${-half_track_width} ${-body_height/2}" rpy="0 0 0" />
         <axis xyz="0 0 1" />
-        <limit upper="${max_steering_angle}" lower="${-max_steering_angle}" effort="10.0" velocity="5.0" />
+        <limit upper="${max_steering_angle}" lower="${-max_steering_angle}" effort="10.0" velocity="2.0" />
+        <dynamics damping="0.1" friction="0.1"/>
     </joint>
     <!-- ================================ -->
@@ -183,5 +197,5 @@
     <link name="fr_right_wheel_link">
         <inertial>
-            <origin xyz="0 0 0" rpy="0 0 0" />
+            <origin xyz="0 0 0" rpy="${pi/2} 0 0" />
             <mass value="${wheel_mass}" />
             <inertia
@@ -193,5 +207,5 @@
         </inertial>
         <visual>
-            <origin xyz="0 0 0" rpy="0 0 0" />
+            <origin xyz="0 0 0" rpy="${pi/2} 0 0" />
             <geometry>
                 <cylinder radius="${wheel_radius}" length="${wheel_thickness}" />
@@ -202,5 +216,5 @@
         </visual>
         <collision>
-            <origin xyz="0 0 0" rpy="0 0 0" />
+            <origin xyz="0 0 0" rpy="${pi/2} 0 0" />
             <geometry>
                 <cylinder radius="${wheel_radius}" length="${wheel_thickness}" />
@@ -211,8 +225,8 @@
         <parent link="fr_right_steer_link" />
         <child link="fr_right_wheel_link" />
-        <origin xyz="0 0 0" rpy="${-pi/2} 0 0" />
-        <axis xyz="0 0 1" />
-        <dynamics friction="0.8" damping="0.5" />
-        <limit lower="-3.14159" upper="3.14159" effort="70" velocity="-1" />
+        <origin xyz="0 0 0" rpy="0 0 0" />
+        <axis xyz="0 1 0" />
+        <dynamics friction="0.1" damping="0.1" />
+        <limit lower="-3.14159" upper="3.14159" effort="70" velocity="50" />
     </joint>
     <!-- ================================ -->
@@ -221,5 +235,5 @@
     <link name="re_left_wheel_link">
         <inertial>
-            <origin xyz="0 0 0" rpy="0 0 0" />
+            <origin xyz="0 0 0" rpy="${pi/2} 0 0" />
             <mass value="${wheel_mass}" />
             <inertia
@@ -231,5 +245,5 @@
         </inertial>
         <visual>
-            <origin xyz="0 0 0" rpy="0 0 0" />
+            <origin xyz="0 0 0" rpy="${pi/2} 0 0" />
             <geometry>
                 <cylinder radius="${wheel_radius}" length="${wheel_thickness}" />
@@ -240,5 +254,5 @@
         </visual>
         <collision>
-            <origin xyz="0 0 0" rpy="0 0 0" />
+            <origin xyz="0 0 0" rpy="${pi/2} 0 0" />
             <geometry>
                 <cylinder radius="${wheel_radius}" length="${wheel_thickness}" />
@@ -249,8 +263,8 @@
         <parent link="chassis_link" />
         <child link="re_left_wheel_link" />
-        <origin xyz="${rear_axle_offset} ${half_track_width} ${-body_height/2}" rpy="${pi/2} 0 0" />
-        <axis xyz="0 0 -1" />
-        <dynamics friction="0.8" damping="0.5" />
-        <limit lower="-3.14159" upper="3.14159" effort="70" velocity="-1" />
+        <origin xyz="${rear_axle_offset} ${half_track_width} ${-body_height/2}" rpy="0 0 0" />
+        <axis xyz="0 1 0" />
+        <dynamics friction="0.1" damping="0.1" />
+        <limit lower="-3.14159" upper="3.14159" effort="70" velocity="50" />
     </joint>
     <!-- ================================ -->
@@ -259,5 +273,5 @@
     <link name="re_right_wheel_link">
         <inertial>
-            <origin xyz="0 0 0" rpy="0 0 0" />
+            <origin xyz="0 0 0" rpy="${pi/2} 0 0" />
             <mass value="${wheel_mass}" />
             <inertia
@@ -269,5 +283,5 @@
         </inertial>
         <visual>
-            <origin xyz="0 0 0" rpy="0 0 0" />
+            <origin xyz="0 0 0" rpy="${pi/2} 0 0" />
             <geometry>
                 <cylinder radius="${wheel_radius}" length="${wheel_thickness}" />
@@ -278,5 +292,5 @@
         </visual>
         <collision>
-            <origin xyz="0 0 0" rpy="0 0 0" />
+            <origin xyz="0 0 0" rpy="${pi/2} 0 0" />
             <geometry>
                 <cylinder radius="${wheel_radius}" length="${wheel_thickness}" />
@@ -287,8 +301,8 @@
         <parent link="chassis_link" />
         <child link="re_right_wheel_link" />
-        <origin xyz="${rear_axle_offset} ${-half_track_width} ${-body_height/2}" rpy="${-pi/2} 0 0" />
-        <axis xyz="0 0 1" />
-        <dynamics friction="0.8" damping="0.5" />
-        <limit lower="-3.14159" upper="3.14159" effort="70" velocity="-1" />
+        <origin xyz="${rear_axle_offset} ${-half_track_width} ${-body_height/2}" rpy="0 0 0" />
+        <axis xyz="0 1 0" />
+        <dynamics friction="0.1" damping="0.1" />
+        <limit lower="-3.14159" upper="3.14159" effort="70" velocity="50" />
     </joint>
     <!-- ================================ -->
@@ -360,9 +374,9 @@
     <!-- Chassis -->
     <gazebo reference="chassis_link">
-        <mu1>0.5</mu1>
-        <mu2>0.5</mu2>
+        <mu1>0.001</mu1>
+        <mu2>0.001</mu2>
         <material>Gazebo/Grey</material>
     </gazebo>
-    <!-- Steering links -->
+    <!-- Steering links
     <gazebo reference="fr_left_steer_link">
         <mu1>0.1</mu1>
@@ -375,24 +389,25 @@
         <material>Gazebo/Black</material>
     </gazebo>
+     -->
     <!-- Front wheels -->
     <gazebo reference="fr_left_wheel_link">
-        <mu1>1.5</mu1>
-        <mu2>1.5</mu2>
+        <mu1>1.0</mu1>
+        <mu2>1.0</mu2>
         <material>Gazebo/DarkGrey</material>
     </gazebo>
     <gazebo reference="fr_right_wheel_link">
-        <mu1>1.5</mu1>
-        <mu2>1.5</mu2>
+        <mu1>1.0</mu1>
+        <mu2>1.0</mu2>
         <material>Gazebo/DarkGrey</material>
     </gazebo>
     <!-- Rear wheels -->
     <gazebo reference="re_left_wheel_link">
-        <mu1>1.5</mu1>
-        <mu2>1.5</mu2>
+        <mu1>1.0</mu1>
+        <mu2>1.0</mu2>
         <material>Gazebo/DarkGrey</material>
     </gazebo>
     <gazebo reference="re_right_wheel_link">
-        <mu1>1.5</mu1>
-        <mu2>1.5</mu2>
+        <mu1>1.0</mu1>
+        <mu2>1.0</mu2>
         <material>Gazebo/DarkGrey</material>
     </gazebo>
@@ -448,35 +463,53 @@
         </plugin>
     </gazebo>
-    <!-- ================================ -->
-    <!-- ACKERMANN DRIVE PLUGIN -->
-    <!-- ================================ -->
+        <!-- Gazebo Control -->
+    <ros2_control name="control" type="system">
+        <hardware>
+            <plugin>gz_ros2_control/GazeboSimSystem</plugin>
+        </hardware>
+        <joint name="fr_left_steer_joint">
+            <command_interface name="position">
+                <!-- <param name="min">${-max_steering_angle}</param>
+                <param name="max">${max_steering_angle}</param> -->
+            </command_interface>
+            <state_interface name="position"/>
+            <state_interface name="velocity"/>
+            <state_interface name="effort"/>
+        </joint>
+        <joint name="fr_right_steer_joint">
+            <command_interface name="position">
+                <!-- <param name="min">${-max_steering_angle}</param>
+                <param name="max">${max_steering_angle}</param> -->
+            </command_interface>
+            <state_interface name="position"/>
+            <state_interface name="velocity"/>
+            <state_interface name="effort"/>
+        </joint>
+        <joint name="re_left_wheel_joint">
+            <command_interface name="velocity">
+                <!-- <param name="min">${-max_wheel_angular_velocity}</param>
+                <param name="max">${max_wheel_angular_velocity}</param> -->
+            </command_interface>
+            <state_interface name="position"/>
+            <state_interface name="velocity"/>
+            <state_interface name="effort"/>
+        </joint>
+        <joint name="re_right_wheel_joint">
+            <command_interface name="velocity">
+                <!-- <param name="min">${-max_wheel_angular_velocity}</param>
+                <param name="max">${max_wheel_angular_velocity}</param> -->
+            </command_interface>
+            <state_interface name="position"/>
+            <state_interface name="velocity"/>
+            <state_interface name="effort"/>
+        </joint>
+    </ros2_control>
     <gazebo>
-        <plugin filename="gz-sim-ackermann-steering-system"
-            name="gz::sim::systems::AckermannSteering">
-            <!-- Wheel joints -->
-            <left_joint>fr_left_wheel_joint</left_joint>
-            <left_joint>re_left_wheel_joint</left_joint>
-            <right_joint>fr_right_wheel_joint</right_joint>
-            <right_joint>re_right_wheel_joint</right_joint>
-            <!-- Steering joints -->
-            <left_steering_joint>fr_left_steer_joint</left_steering_joint>
-            <right_steering_joint>fr_right_steer_joint</right_steering_joint>
-            <steering_joint>virtual_steering_wheel_joint</steering_joint>
-            <!-- Wheel parameters -->
-            <wheel_separation>${track_width}</wheel_separation>
-            <kingpin_width>${track_width}</kingpin_width>
-            <wheel_base>${wheelbase}</wheel_base>
-            <wheel_radius>${wheel_radius}</wheel_radius>
-            <min_velocity>-1</min_velocity>
-            <max_velocity>1</max_velocity>
-            <!-- Steering limits -->
-            <steering_limit>${max_steering_angle}</steering_limit>
-            <!-- Command and odometry topics -->
-            <topic>/cmd_vel</topic>
-            <tf_topic>/tf</tf_topic>
-            <odom_topic>/odom</odom_topic>
-            <frame_id>odom</frame_id>
-            <child_frame_id>base_footprint</child_frame_id>
-            <odom_publish_frequency>50</odom_publish_frequency>
+        <plugin filename="gz_ros2_control-system" name="gz_ros2_control::GazeboSimROS2ControlPlugin">
+            <parameters> $(find ackermann_gazebo)/config/gz_ros2_control.yaml</parameters>
+            <ros>
+                <remapping>ackermann_steering_controller/tf_odometry:=/tf</remapping>
+                <remapping>ackermann_steering_controller/odometry:=/odom</remapping>
+            </ros>
         </plugin>
     </gazebo>

File: src/ackermann_gazebo/urdf/gz_ackermann_core.xacro (robot description, xacro)
@@ -126,6 +126,6 @@
         </plugin>
     </gazebo>
-    <!-- ================================ -->
-    <!-- ACKERMANN DRIVE PLUGIN -->
+    <!-- ================================
+    <! ACKERMANN DRIVE PLUGIN -->
     <!-- ================================ -->
     <gazebo>
@@ -134,7 +134,7 @@
             <!-- Wheel joints -->
             <left_joint>fr_left_wheel_joint</left_joint>
+            <left_joint>re_left_wheel_joint</left_joint>
             <right_joint>fr_right_wheel_joint</right_joint>
-            <left_rear_joint>re_left_wheel_joint</left_rear_joint>
-            <right_rear_joint>re_right_wheel_joint</right_rear_joint>
+            <right_joint>re_right_wheel_joint</right_joint>
             <!-- Steering joints -->
             <left_steering_joint>fr_left_steer_joint</left_steering_joint>
@@ -142,20 +142,19 @@
             <steering_joint>virtual_steering_wheel_joint</steering_joint>
             <!-- Wheel parameters -->
-            <wheel_separation>0.504</wheel_separation>
-            <kingpin_width>0.49238</kingpin_width>
-            <wheel_base>0.54838</wheel_base>
-            <wheel_radius>0.14</wheel_radius>
+            <wheel_separation>${track_width}</wheel_separation>
+            <kingpin_width>${track_width}</kingpin_width>
+            <wheel_base>${wheelbase}</wheel_base>
+            <wheel_radius>${wheel_radius}</wheel_radius>
+            <min_velocity>-1</min_velocity>
+            <max_velocity>1</max_velocity>
             <!-- Steering limits -->
-            <max_steer>0.383972</max_steer>
-            <max_steering_angle>1.570796</max_steering_angle>
+            <steering_limit>${max_steering_angle}</steering_limit>
             <!-- Command and odometry topics -->
             <topic>/cmd_vel</topic>
+            <tf_topic>/tf</tf_topic>
             <odom_topic>/odom</odom_topic>
-            <odom_frame>odom</odom_frame>
-            <robot_base_frame>base_footprint</robot_base_frame>
-            <!-- Publishing options -->
-            <publish_odom>true</publish_odom>
-            <publish_odom_tf>true</publish_odom_tf>
-            <publish_wheel_tf>false</publish_wheel_tf>
+            <frame_id>odom</frame_id>
+            <child_frame_id>base_footprint</child_frame_id>
+            <odom_publish_frequency>50</odom_publish_frequency>
         </plugin>
     </gazebo>
