Commit message: start navigation

File: src/ackermann_gazebo/urdf/bot_sample.xacro (robot description, xacro)
@@ -5,7 +5,7 @@
     <!-- ================================ -->
     <xacro:property name="body_mass" value="1.58" />
-    <xacro:property name="body_length" value="0.475" />
+    <xacro:property name="body_length" value="0.460" />
     <xacro:property name="body_width" value="0.21" />
-    <xacro:property name="body_height" value="0.160" />
+    <xacro:property name="body_height" value="0.110" />
     <xacro:property name="wheelbase" value="0.285" />
     <xacro:property name="track_width" value="0.280" />
@@ -340,5 +340,5 @@
         <child link="bot_ackermann/base_footprint/gpu_lidar" />
         <!-- LiDAR at front edge + its radius, sitting on top surface -->
-        <origin xyz=" 0.1 0.0 ${body_height/2 + lidar_height/2}" rpy="0 0 0" />
+        <origin xyz=" 0.15 0.0 ${body_height/2 + lidar_height/2}" rpy="0 0 0" />
     </joint>
     <!-- ================================ -->
@@ -463,53 +463,35 @@
         </plugin>
     </gazebo>
-        <!-- Gazebo Control -->
-    <ros2_control name="control" type="system">
-        <hardware>
-            <plugin>gz_ros2_control/GazeboSimSystem</plugin>
-        </hardware>
-        <joint name="fr_left_steer_joint">
-            <command_interface name="position">
-                <!-- <param name="min">${-max_steering_angle}</param>
-                <param name="max">${max_steering_angle}</param> -->
-            </command_interface>
-            <state_interface name="position"/>
-            <state_interface name="velocity"/>
-            <state_interface name="effort"/>
-        </joint>
-        <joint name="fr_right_steer_joint">
-            <command_interface name="position">
-                <!-- <param name="min">${-max_steering_angle}</param>
-                <param name="max">${max_steering_angle}</param> -->
-            </command_interface>
-            <state_interface name="position"/>
-            <state_interface name="velocity"/>
-            <state_interface name="effort"/>
-        </joint>
-        <joint name="re_left_wheel_joint">
-            <command_interface name="velocity">
-                <!-- <param name="min">${-max_wheel_angular_velocity}</param>
-                <param name="max">${max_wheel_angular_velocity}</param> -->
-            </command_interface>
-            <state_interface name="position"/>
-            <state_interface name="velocity"/>
-            <state_interface name="effort"/>
-        </joint>
-        <joint name="re_right_wheel_joint">
-            <command_interface name="velocity">
-                <!-- <param name="min">${-max_wheel_angular_velocity}</param>
-                <param name="max">${max_wheel_angular_velocity}</param> -->
-            </command_interface>
-            <state_interface name="position"/>
-            <state_interface name="velocity"/>
-            <state_interface name="effort"/>
-        </joint>
-    </ros2_control>
+     <!-- ================================
+    <! ACKERMANN DRIVE PLUGIN -->
+    <!-- ================================ -->
     <gazebo>
-        <plugin filename="gz_ros2_control-system" name="gz_ros2_control::GazeboSimROS2ControlPlugin">
-            <parameters> $(find ackermann_gazebo)/config/gz_ros2_control.yaml</parameters>
-            <ros>
-                <remapping>ackermann_steering_controller/tf_odometry:=/tf</remapping>
-                <remapping>ackermann_steering_controller/odometry:=/odom</remapping>
-            </ros>
+        <plugin filename="gz-sim-ackermann-steering-system"
+            name="gz::sim::systems::AckermannSteering">
+            <!-- Wheel joints -->
+            <left_joint>fr_left_wheel_joint</left_joint>
+            <left_joint>re_left_wheel_joint</left_joint>
+            <right_joint>fr_right_wheel_joint</right_joint>
+            <right_joint>re_right_wheel_joint</right_joint>
+            <!-- Steering joints -->
+            <left_steering_joint>fr_left_steer_joint</left_steering_joint>
+            <right_steering_joint>fr_right_steer_joint</right_steering_joint>
+            <steering_joint>virtual_steering_wheel_joint</steering_joint>
+            <!-- Wheel parameters -->
+            <wheel_separation>${track_width}</wheel_separation>
+            <kingpin_width>${track_width}</kingpin_width>
+            <wheel_base>${wheelbase}</wheel_base>
+            <wheel_radius>${wheel_radius}</wheel_radius>
+            <min_velocity>-1</min_velocity>
+            <max_velocity>1</max_velocity>
+            <!-- Steering limits -->
+            <steering_limit>${max_steering_angle}</steering_limit>
+            <!-- Command and odometry topics -->
+            <topic>/cmd_vel</topic>
+            <tf_topic>/tf</tf_topic>
+            <odom_topic>/odom</odom_topic>
+            <frame_id>odom</frame_id>
+            <child_frame_id>base_footprint</child_frame_id>
+            <odom_publish_frequency>50</odom_publish_frequency>
         </plugin>
     </gazebo>
@@ -518,4 +500,4 @@
             <render_engine>ogre2</render_engine>
         </plugin>
-  </gazebo>
+    </gazebo>
 </robot>
